Commit message: test: co: xacro: Add collision values to the joints
Signed-off-by: Pallav Joshi <pallav.joshi@amd.com>

File: test/ros2_co_control/urdf/motor_kit.xacro (robot description, xacro)
@@ -10,4 +10,12 @@
             </material>
         </visual>
+        <collision>
+            <geometry>
+                <box size="0.8 1.6 0.1"/>
+            </geometry>
+            <material name="White">
+                <color rgba="1 1 1 1"/>
+            </material>
+        </collision>
     </link>
     <joint name="motor_joint" type="fixed">
@@ -26,4 +34,13 @@
             </material>
         </visual>
+        <collision>
+            <geometry>
+                <cylinder length="0.4" radius="0.1"/>
+            </geometry>
+            <origin rpy="1.57075 0 0" xyz="0 0 0.15"/>
+            <material name="Black">
+                <color rgba="0.2 0.2 0.2 1"/>
+            </material>
+        </collision>
     </link>
     <joint name="screw_joint" type="fixed">
@@ -42,4 +59,13 @@
             </material>
         </visual>
+        <collision>
+            <geometry>
+                <cylinder length="0.04" radius="0.01"/>
+            </geometry>
+            <origin rpy="1.57075 0 0" xyz="0 0 0.15"/>
+            <material name="Grey">
+                <color rgba="0.9 0.9 0.9 1"/>
+            </material>
+        </collision>
     </link>
     <joint name="wheel_joint" type="continuous">
@@ -58,4 +84,12 @@
             </material>
         </visual>
+        <collision>
+            <geometry>
+                <cylinder length="0.04" radius="0.125"/>
+            </geometry>
+            <material name="Grey">
+                <color rgba="0.9 0.9 0.9 1"/>
+            </material>
+        </collision>
     </link>
 </robot>
