Commit message: test: ros2_control: Update the device and controller
- Update bus configuration for ros2_co_control.
- Use kd240_wheel as the device name for the driver invocation.
- Add profile_velocity_mode as the type of velocity_mode
- Use only one joint and rename it to wheel_joint
- Add velocity command interface to the wheel_joint
- Add position state interface to the wheel_joint
- Remove forward controller with velocity controller

Signed-off-by: Pallav Joshi <pallav.joshi@amd.com>

File: test/ros2_co_control/urdf/kd240.urdf.xacro (robot description, xacro)
@@ -3,3 +3,10 @@
     <xacro:include filename="motor_kit.xacro" />
     <xacro:include filename="ros2_control.xacro" />
+    <xacro:define_control
+        name="foc_system"
+        prefix=""
+        bus_config="$(find ros2_co_control)/config/motor_control/bus.yml"
+        master_config="$(find ros2_co_control)/config/motor_control/master.dcf"
+        can_interface_name="can0"
+        master_bin="" />
 </robot>

File: test/ros2_co_control/urdf/ros2_control.xacro (robot description, xacro)
@@ -16,18 +16,11 @@
               <param name="master_bin">"${master_bin}"</param>
             </hardware>
-            <joint name="${prefix}joint1">
-                <param name="device_name">wheel_joint</param>
+            <joint name="wheel_joint">
+                <param name="device_name">kd240_wheel</param>
+                <state_interface name="velocity" />
+                <state_interface name="position" />
                 <command_interface name="velocity" />
-                <state_interface name="position" />
-                <state_interface name="velocity" />
             </joint>
         </ros2_control>
     </xacro:macro>
-    <xacro:define_control
-        name="foc_system"
-        prefix=""
-        bus_config="$(find ros2_co_control)/config/motor_control/bus.yml"
-        master_config="$(find ros2_co_control)/config/motor_control/master.dcf"
-        can_interface_name="vcan0"
-        master_bin="" />
 </robot>
